File: Advanced_PCB.kicad_sch (KiCad schematic)
At the start: 0 parts

Commit message: finish usb-c charger for now
Parts:
- added C1: 0u1, symbol Device:C
- added F1: 0ZCH0110AF2E, FUSC3226X100N, symbol 0ZCH0110AF2E:0ZCH0110AF2E
- added J1: SS-52400-002, SS-52400-002:BELFUSE_SS-52400-002, symbol SS-52400-002:SS-52400-002
- added J2: B2B-PH-SM4-TB, B2B-PH-SM4-TB:JST_B2B-PH-SM4-TB, symbol B2B-PH-SM4-TB:B2B-PH-SM4-TB
- added LED1: LTST-C170KRKT, LEDC2012X120N, symbol LTST-C170KRKT:LTST-C170KRKT
- added LED2: LTST-C170GKT, LEDC2012X120N, symbol LTST-C170GKT:LTST-C170GKT
- added LED3: LTST-C170TBKT, LEDC2012X120N, symbol LTST-C170TBKT:LTST-C170TBKT
- added R1, R2: 10K, symbol Device:R
- added R3, R4: 5k1, symbol Device:R
- added R5, R6: 2k, symbol Device:R
- added R7, R8, R9: 470R, symbol Device:R
- added U1: MCP73871-2CAI_ML, MCP73871-2CAI_ML:QFN50P400X400X100-21N, symbol MCP73871-2CAI_ML:MCP73871-2CAI_ML
- added VR1: LM1117MPX-3.3, LM1117MPX-3.3:VREG_LM1117MPX-3.3, symbol LM1117MPX-3.3:LM1117MPX-3.3
Connections:
- new net: J1.A5 (CC1), R4.1
- new net: LED1.1 (K), R9.2
- new net: LED1.2 (A), LED2.2 (A), LED3.2 (A)
- new net: LED2.1 (K), R8.2
- new net: R5.2, U1.12 (PROG3)
- new net: U1.1 (OUT), U1.20 (OUT)
- new net: U1.10 (VSS), U1.11 (VSS), U1.21 (VSS)
- new net: R6.2, U1.13 (PROG1)
- new net: U1.14 (VBAT), U1.15 (VBAT)
- new net: U1.18 (IN), U1.19 (IN)
- new net: R2.1, U1.5 (THERM)
- new net: R9.1, U1.6 (~{PG})
- new net: R8.1, U1.7 (STAT2)
- new net: R7.1, U1.8 (STAT1/~{LBO})
- new net: R1.2, U1.9 (~{TE})
- new net: LED3.1 (K), R7.2
- new net: J1.B5 (CC2), R3.1
- new net +5V_USB: F1.2
- new net GND: C1.2, J1.A1 (GNDA1), J1.A12 (GNDA2), J1.B1 (GNDB1), J1.B12 (GNDB2), J1.G1 (GND/SHIELD), J1.G2 (GND/SHIELD), J1.G3 (GND/SHIELD), J1.G4 (GND/SHIELD), J1.S1 (GND/SHIELD), J1.S2 (GND/SHIELD), J1.S3 (GND/SHIELD), J1.S4 (GND/SHIELD), R1.1, R2.2, R3.2, R4.2, R5.1, R6.1
- new net USB_DN: J1.A7 (DN1), J1.B7 (DN2)
- new net USB_DP: J1.A6 (DP1), J1.B6 (DP2)
- new net VBUS: C1.1, F1.1, J1.A4 (VBUSA1), J1.A9 (VBUSA2), J1.B4 (VBUSB1), J1.B9 (VBUSB2)
- no-connect marks 0 -> 10
Other:
- note added: "Battery connector"
- note added: "Li-Po battery charger"
- note added: "USB-C Connector"
- note added: "Voltage regulator"
- title: (none) -> ESP32 sensor board
